File: triggerbox.sch (EAGLE design)
At the start: 19 parts, among them IC1 LM311N, IC2 4027D, Q1 BS170, Q2 BS170, Q3 BS170

Commit message: schematic triggerbox2
Parts:
- removed LED2: red, led:LED5MM
- removed LED3: green, led:LED5MM
- removed PAD1: trigger-in, wirepad:WIREPAD1,6/0,8
- removed PAD2: pc-parallel, wirepad:WIREPAD1,6/0,8
- removed PAD3: WIREPAD1,6/0,8, wirepad:WIREPAD1,6/0,8
- added BIOSEMI-8, PC-RESET, TRIGGER: WIREPAD1,6/0,8, wirepad:WIREPAD1,6/0,8
- added GREEN, RED: (no value), led:LED5MM
- YELLOW: value Yellow -> (none)
- renumbered LED1 to YELLOW
Connections:
- net N$10: now also RED.A; no longer LED2.A
- net N$11: now also GREEN.A; no longer LED3.A
- net N$12: now also RED.C; no longer LED2.C
- net N$13: now also GREEN.C; no longer LED3.C
- net N$5: now also TRIGGER.P; no longer PAD1.P
- net N$6: now also PC-RESET.P; no longer PAD2.P
- net N$7: now also BIOSEMI-8.P; no longer PAD3.P
Other:
- moved on the sheet: R6, R7, R8

Commit message: schematic triggerbox3
Parts:
- added C1: 1u, rcl:C-EUC0805
Connections:
- net +5V: now also C1.1, IC2P.VDD
- net GND: now also C1.2, IC2A.CLK, IC2A.J, IC2A.K, IC2P.VSS
Other:
- moved on the sheet: PC-RESET
